File: Schematics/DegraderDosimeter/PulseShaper.kicad_sch (KiCad schematic)
At the start: 10 parts, among them J2 Conn_Coaxial, U8 ADA4891-2ARZ-R7

Commit message: Use 1206 for every resistor in the project
The Ethernet sheet was the only one on 0402, set that way to match the
MB1364 BOM. The other four sheets already used
Resistor_SMD:R_1206_3216Metric_Pad1.30x1.75mm_HandSolder, so move the
20 Ethernet resistors to the same footprint. All 37 resistors in the
project now share one package, which suits hand assembly.

This deviates from the ST reference for the eight resistors on the
high-speed nets: R3-R6 (33R RMII series) and R12-R15 (49R9 centre-tap
terminations). 1206 has more parasitic inductance and larger pads than
the 0402 parts ST fits. 100BASE-TX is tolerant enough that this should
still work, but 0402 would be the better choice on those eight.

This commit also captures schematic edits made in KiCad outside this
session: a project-wide re-annotation and the removal of R21/R22, the
two 75R resistors that terminated the jack's unused pairs.

Co-Authored-By: Claude Opus 5 <noreply@anthropic.com>
Claude-Session: https://claude.ai/code/session_01Ej9hevrS5JU2uwVi6UHQUS
Parts:
- renumbered C27 to C45, C26 to C46, R28 to R27, R29 to R28, R30 to R29, R31 to R30, R33 to R31
