File: Schematics/DegraderDosimeter/PulseShaper.kicad_sch (KiCad schematic)
At the start: 10 parts, among them J2 Conn_Coaxial, U8 ADA4891-2ARZ-R7

Commit message: Bring the DegraderDosimeter schematic up to a routable state
Single ECAD commit on top of "First upload", carrying both the earlier
board-bring-up work and this session's changes. Squashed here so the
schematic history is separate from the FirmwareUpdate restructure, which
stays on main.

Library resolution
  Register the A4988 and LM60430DRPKR symbol libraries in sym-lib-table,
  and the DE15, DRIVER-A4988SETTR-T_QFN28_ and KRJ-CB4.2GYZNL footprint
  libraries in fp-lib-table. Point H1102NL at ${KIPRJMOD} instead of the
  undefined ${CUSTOM}. All 26 symbols and 24 footprints now resolve.

Degrader to MCU
  Wire all 32 degrader signals to the STM32H723: 11 A4988/L293D controls
  and 21 lens limit switches. Reuse the F746 firmware's pin assignment
  where it does not clash with the dosimeter; MS1 and MS2 move to PD14
  and PD15 because PD11/PD12 are pulse-capture pins, and !ENABLE takes
  PB7 as the firmware never assigned it. Grow the MCU_H723 sheet so its
  right edge spans the Degrader sheet, giving one straight wire per net.

Net naming and classes
  Drop the duplicate port label on the 50 pins that already carry a
  functional hierarchical label, so nets read STEP/MS1/RMII_REF_CLK
  rather than PD14/PA1; unused pins keep their port label and bus. Name
  the remaining 73 auto-named nets. Add ETH_DIFF_100R, ETH_RMII, POWER,
  MOTOR and ANALOG net classes. The four MDI pairs get 0.15 mm track on
  a 0.30 mm gap, which is 100 ohm differential on the declared stackup
  (F.Cu over In1.Cu, 0.1 mm prepreg, er 4.5) - reconfirm if the fab
  ships a different stackup.

Connection fixes
  - MDC/MDIO were crossed: PA2 landed on the PHY's MDC pin and PC1 on
    MDIO. Swapped the two labels in Ethernet.kicad_sch.
  - PULSE_6 moved PD11 -> PD12, the TIM4_CH1 pin BLM_Code.ioc expects.
  - PulseShaper 1, 2 and 5 outputs missed their sheet pins by 2-81 um.
  - XTAL1 stopped 0.254 mm short of Y1/C1, leaving the PHY crystal open.
  - C32/C35 and C39/C40, the U5 and U7 cap returns, h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
Parts:
- added TP1, TP13, TP19, TP7: PulseInput, TestPoint:TestPoint_Pad_D2.5mm, symbol Connector:TestPoint
- added TP25: PulseOut, TestPoint:TestPoint_Pad_D2.5mm, symbol Connector:TestPoint
- renumbered C27 to C45, C26 to C46, R28 to R27, R29 to R28, R30 to R29, R31 to R30, R33 to R31
Connections:
- net STAGE2_FB: now reaches R30.2, RV1.1, U8.P$6
- net STAGE2_FB: now also TP19.1
- net STAGE1_FB: now reaches R27.2, R28.1, U8.P$2
- net STAGE2_IN: now reaches R29.2, R31.1, U8.P$5
- net STAGE2_IN: now also TP13.1
- net PULSE_IN: now reaches J2.1 (In), U8.P$3
- net PULSE_IN: now also TP1.1
- net STAGE1_OUT: now reaches R28.2, R29.1, U8.P$1
- net STAGE1_OUT: now also TP7.1
- net pulse_out1 renamed pulse_out
- net pulse_out: now also TP25.1
