File: Schematics/DegraderDosimeter/Degrader.kicad_sch (KiCad schematic)
At the start: 17 parts, among them J2 DE15_Socket_HighDensity, J3 DE15_Socket_HighDensity, U8 DRIVER-A4988SETTR-T_QFN28_

Commit message: Use 1206 for every resistor in the project
The Ethernet sheet was the only one on 0402, set that way to match the
MB1364 BOM. The other four sheets already used
Resistor_SMD:R_1206_3216Metric_Pad1.30x1.75mm_HandSolder, so move the
20 Ethernet resistors to the same footprint. All 37 resistors in the
project now share one package, which suits hand assembly.

This deviates from the ST reference for the eight resistors on the
high-speed nets: R3-R6 (33R RMII series) and R12-R15 (49R9 centre-tap
terminations). 1206 has more parasitic inductance and larger pads than
the 0402 parts ST fits. 100BASE-TX is tolerant enough that this should
still work, but 0402 would be the better choice on those eight.

This commit also captures schematic edits made in KiCad outside this
session: a project-wide re-annotation and the removal of R21/R22, the
two 75R resistors that terminated the jack's unused pairs.

Co-Authored-By: Claude Opus 5 <noreply@anthropic.com>
Claude-Session: https://claude.ai/code/session_01Ej9hevrS5JU2uwVi6UHQUS
Parts:
- renumbered C29 to C57, C28 to C58, C30 to C59, C33 to C60, C26 to C61, C31 to C62, C27 to C63, C32 to C64, J2 to J8, J3 to J9, R28 to R57, R31 to R58, R29 to R59, R32 to R60, R33 to R61, R30 to R62, U8 to U14
Changed lines of the file:
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@@
 		(dnp no)
 		(fields_autoplaced yes)
-		(property "Reference" "C30"
+		(property "Reference" "C59"
 			(at 256.54 170.9419 0)
 			(show_name no)
@@
 			(project "DegraderDosimeter"
 				(path "/f3c83d46-b432-4960-ae55-27eb620ca6d0/9ad00133-e13c-465e-ad59-297593e6d3f6"
-					(reference "C30")
+					(reference "C59")
 					(unit 1)
 				)
@@
 		(in_pos_files yes)
 		(dnp no)
-		(property "Reference" "R33"
+		(property "Reference" "R61"
 			(at 332.486 171.196 0)
 			(show_name no)
@@
 			(project "DegraderDosimeter"
 				(path "/f3c83d46-b432-4960-ae55-27eb620ca6d0/9ad00133-e13c-465e-ad59-297593e6d3f6"
-					(reference "R33")
+					(reference "R61")
 					(unit 1)
 				)
@@
 		(dnp no)
 		(fields_autoplaced yes)
-		(property "Reference" "#PWR028"
+		(property "Reference" "#PWR087"
 			(at 331.978 205.74 0)
 			(hide yes)
@@
 			(project "DegraderDosimeter"
 				(path "/f3c83d46-b432-4960-ae55-27eb620ca6d0/9ad00133-e13c-465e-ad59-297593e6d3f6"
-					(reference "#PWR028")
+					(reference "#PWR087")
 					(unit 1)
 				)
@@
 		(in_pos_files yes)
 		(dnp no)
-		(property "Reference" "R29"
+		(property "Reference" "R59"
 			(at 302.006 120.142 90)
 			(show_name no)
@@
 			(project "DegraderDosimeter"
 				(path "/f3c83d46-b432-4960-ae55-27eb620ca6d0/9ad00133-e13c-465e-ad59-297593e6d3f6"
-					(reference "R29")
+					(reference "R59")
 					(unit 1)
 				)
@@
 		(in_pos_files yes)
 		(dnp no)
-		(property "Reference" "R30"
+		(property "Reference" "R62"
 			(at 345.948 168.402 90)
 			(show_name no)
@@
 			(project "DegraderDosimeter"
 				(path "/f3c83d46-b432-4960-ae55-27eb620ca6d0/9ad00133-e13c-465e-ad59-297593e6d3f6"
-					(reference "R30")
+					(reference "R62")
 					(unit 1)
 				)
@@
 		(dnp no)
 		(fields_autoplaced yes)
-		(property "Reference" "C32"
+		(property "Reference" "C64"
 			(at 340.36 187.4519 0)
 			(show_name no)
@@
 			(project "DegraderDosimeter"
 				(path "/f3c83d46-b432-4960-ae55-27eb620ca6d0/9ad00133-e13c-465e-ad59-297593e6d3f6"
-					(reference "C32")
+					(reference "C64")
 					(unit 1)
 				)
@@
 		(dnp no)
 		(fields_autoplaced yes)
-		(property "Reference" "#PWR026"
+		(property "Reference" "#PWR081"
 			(at 264.668 148.336 0)
 			(hide yes)
@@
 			(project "DegraderDosimeter"
 				(path "/f3c83d46-b432-4960-ae55-27eb620ca6d0/9ad00133-e13c-465e-ad59-297593e6d3f6"
-					(reference "#PWR026")
+					(reference "#PWR081")
 					(unit 1)
 				)
@@
 		(dnp no)
 		(fields_autoplaced yes)
-		(property "Reference" "#PWR031"
+		(property "Reference" "#PWR085"
 			(at 308.864 213.36 0)
 			(hide yes)
@@
 			(project "DegraderDosimeter"
 				(path "/f3c83d46-b432-4960-ae55-27eb620ca6d0/9ad00133-e13c-465e-ad59-297593e6d3f6"
-					(reference "#PWR031")
+					(reference "#PWR085")
 					(unit 1)
 				)
@@
 		(dnp no)
 		(fields_autoplaced yes)
-		(property "Reference" "C28"
+		(property "Reference" "C58"
 			(at 248.92 140.9699 0)
 			(show_name no)
@@
 			(project "DegraderDosimeter"
 				(path "/f3c83d46-b432-4960-ae55-27eb620ca6d0/9ad00133-e13c-465e-ad59-297593e6d3f6"
-					(reference "C28")
+					(reference "C58")
 					(unit 1)
 				)
@@
 		(in_pos_files yes)
 		(dnp no)
-		(property "Reference" "C27"
+		(property "Reference" "C63"
 			(at 332.994 128.016 0)
 			(show_name no)
@@
 			(project "DegraderDosimeter"
 				(path "/f3c83d46-b432-4960-ae55-27eb620ca6d0/9ad00133-e13c-465e-ad59-297593e6d3f6"
-					(reference "C27")
+					(reference "C63")
 					(unit 1)
 				)
@@
 		(dnp no)
 		(fields_autoplaced yes)
-		(property "Reference" "C33"
+		(property "Reference" "C60"
 			(at 285.75 198.3739 0)
 			(show_name no)
@@
 			(project "DegraderDosimeter"
 				(path "/f3c83d46-b432-4960-ae55-27eb620ca6d0/9ad00133-e13c-465e-ad59-297593e6d3f6"
-					(reference "C33")
+					(reference "C60")
 					(unit 1)
 				)
@@
 		(dnp no)
 		(fields_autoplaced yes)
-		(property "Reference" "#PWR027"
+		(property "Reference" "#PWR089"
 			(at 354.076 174.244 0)
 			(hide yes)
@@
 			(project "DegraderDosimeter"
 				(path "/f3c83d46-b432-4960-ae55-27eb620ca6d0/9ad00133-e13c-465e-ad59-297593e6d3f6"
-					(reference "#PWR027")
+					(reference "#PWR089")
 					(unit 1)
 				)
@@
 		(in_pos_files yes)
 		(dnp no)
-		(property "Reference" "R28"
+		(property "Reference" "R57"
 			(at 277.876 119.888 90)
 			(show_name no)
@@
 			(project "DegraderDosimeter"
 				(path "/f3c83d46-b432-4960-ae55-27eb620ca6d0/9ad00133-e13c-465e-ad59-297593e6d3f6"
-					(reference "R28")
+					(reference "R57")
 					(unit 1)
 				)
@@
 		(dnp no)
 		(fields_autoplaced yes)
-		(property "Reference" "#PWR025"
+		(property "Reference" "#PWR088"
 			(at 351.282 134.112 0)
 			(hide yes)
@@
 			(project "DegraderDosimeter"
 				(path "/f3c83d46-b432-4960-ae55-27eb620ca6d0/9ad00133-e13c-465e-ad59-297593e6d3f6"
-					(reference "#PWR025")
+					(reference "#PWR088")
 					(unit 1)
 				)
@@
 		(dnp no)
 		(fields_autoplaced yes)
-		(property "Reference" "#PWR024"
+		(property "Reference" "#PWR080"
 			(at 244.856 154.432 0)
 			(hide yes)
@@
 			(project "DegraderDosimeter"
 				(path "/f3c83d46-b432-4960-ae55-27eb620ca6d0/9ad00133-e13c-465e-ad59-297593e6d3f6"
-					(reference "#PWR024")
+					(reference "#PWR080")
 					(unit 1)
 				)
@@
 		(in_pos_files yes)
 		(dnp no)
-		(property "Reference" "R32"
+		(property "Reference" "R60"
 			(at 312.712 199.216 0)
 			(show_name no)
@@
 			(project "DegraderDosimeter"
 				(path "/f3c83d46-b432-4960-ae55-27eb620ca6d0/9ad00133-e13c-465e-ad59-297593e6d3f6"
-					(reference "R32")
+					(reference "R60")
 					(unit 1)
 				)
@@
 		(in_pos_files yes)
 		(dnp no)
-		(property "Reference" "U8"
+		(property "Reference" "U14"
 			(at 324.358 147.32 0)
 			(show_name no)
@@
 			(project "DegraderDosimeter"
 				(path "/f3c83d46-b432-4960-ae55-27eb620ca6d0/9ad00133-e13c-465e-ad59-297593e6d3f6"
-					(reference "U8")
+					(reference "U14")
 					(unit 1)
 				)
@@
 		(dnp no)
 		(fields_autoplaced yes)
-		(property "Reference" "#PWR023"
+		(property "Reference" "#PWR086"
 			(at 311.404 134.62 0)
 			(hide yes)
@@
 			(project "DegraderDosimeter"
 				(path "/f3c83d46-b432-4960-ae55-27eb620ca6d0/9ad00133-e13c-465e-ad59-297593e6d3f6"
-					(reference "#PWR023")
+					(reference "#PWR086")
 					(unit 1)
 				)
@@
 		(in_pos_files yes)
 		(dnp no)
-		(property "Reference" "C31"
+		(property "Reference" "C62"
 			(at 320.04 187.198 0)
 			(show_name no)
@@
 			(project "DegraderDosimeter"
 				(path "/f3c83d46-b432-4960-ae55-27eb620ca6d0/9ad00133-e13c-465e-ad59-297593e6d3f6"
-					(reference "C31")
+					(reference "C62")
 					(unit 1)
 				)
@@
 		(dnp no)
 		(fields_autoplaced yes)
-		(property "Reference" "#PWR030"
+		(property "Reference" "#PWR084"
 			(at 294.64 213.36 0)
 			(hide yes)
@@
 			(project "DegraderDosimeter"
 				(path "/f3c83d46-b432-4960-ae55-27eb620ca6d0/9ad00133-e13c-465e-ad59-297593e6d3f6"
-					(reference "#PWR030")
+					(reference "#PWR084")
 					(unit 1)
 				)
@@
 		(dnp no)
 		(fields_autoplaced yes)
-		(property "Reference" "J3"
+		(property "Reference" "J9"
 			(at 188.214 238.252 0)
 			(show_name no)
@@
 			(project "DegraderDosimeter"
 				(path "/f3c83d46-b432-4960-ae55-27eb620ca6d0/9ad00133-e13c-465e-ad59-297593e6d3f6"
-					(reference "J3")
+					(reference "J9")
 					(unit 1)
 				)
@@
 		(dnp no)
 		(fields_autoplaced yes)
-		(property "Reference" "#PWR029"
+		(property "Reference" "#PWR083"
 			(at 281.94 212.852 0)
 			(hide yes)
@@
 			(project "DegraderDosimeter"
 				(path "/f3c83d46-b432-4960-ae55-27eb620ca6d0/9ad00133-e13c-465e-ad59-297593e6d3f6"
-					(reference "#PWR029")
+					(reference "#PWR083")
 					(unit 1)
 				)
@@
 		(dnp no)
 		(fields_autoplaced yes)
-		(property "Reference" "#PWR022"
+		(property "Reference" "#PWR082"
 			(at 271.272 133.35 0)
 			(hide yes)
@@
 			(project "DegraderDosimeter"
 				(path "/f3c83d46-b432-4960-ae55-27eb620ca6d0/9ad00133-e13c-465e-ad59-297593e6d3f6"
-					(reference "#PWR022")
+					(reference "#PWR082")
 					(unit 1)
 				)
@@
 		(dnp no)
 		(fields_autoplaced yes)
-		(property "Reference" "C29"
+		(property "Reference" "C57"
 			(at 237.49 163.0679 0)
 			(show_name no)
@@
 			(project "DegraderDosimeter"
 				(path "/f3c83d46-b432-4960-ae55-27eb620ca6d0/9ad00133-e13c-465e-ad59-297593e6d3f6"
-					(reference "C29")
+					(reference "C57")
 					(unit 1)
 				)
@@
 		(in_pos_files yes)
 		(dnp no)
-		(property "Reference" "R31"
+		(property "Reference" "R58"
 			(at 298.704 199.746 0)
 			(show_name no)
@@
 			(project "DegraderDosimeter"
 				(path "/f3c83d46-b432-4960-ae55-27eb620ca6d0/9ad00133-e13c-465e-ad59-297593e6d3f6"
-					(reference "R31")
+					(reference "R58")
 					(unit 1)
 				)
@@
 		(in_pos_files yes)
 		(dnp no)
-		(property "Reference" "C26"
+		(property "Reference" "C61"
 			(at 322.834 127.5079 0)
 			(show_name no)
@@
 			(project "DegraderDosimeter"
 				(path "/f3c83d46-b432-4960-ae55-27eb620ca6d0/9ad00133-e13c-465e-ad59-297593e6d3f6"
-					(reference "C26")
+					(reference "C61")
 					(unit 1)
 				)
@@
 		(dnp no)
 		(fields_autoplaced yes)
-		(property "Reference" "J2"
+		(property "Reference" "J8"
 			(at 92.964 238.506 0)
 			(show_name no)
@@
 			(project "DegraderDosimeter"
 				(path "/f3c83d46-b432-4960-ae55-27eb620ca6d0/9ad00133-e13c-465e-ad59-297593e6d3f6"
-					(reference "J2")
-					(unit 1)
-				)
+					(reference "J8")
+					(unit 1)
+				)

Commit message: Give every footprint pad a symbol pin so no pad is left netless
Updating the PCB warned about eight pads that had no matching symbol
pin, so they would have been placed with no net: U5/U7 pad 4, Y2 pads
3 and 4, and J8/J9 pads 16 and 17. Three separate causes:

SOT-223 tab (U5, U7). The TC1262 tab is electrically the same node as
pin 2, GND; the vendor symbol in Libs/TC1262-3.3VDB draws pins 2 and 4
stacked at one point, which confirms it. Renumber the footprint's tab
pad from 4 to 2 so it inherits GND. No schematic change, and the tab is
the regulator's heat path, so it needs to be connected.

Crystal case (Y2). Same fix already applied to Y1: Device:Crystal on a
4-pad footprint left the two case pads unmapped. Move to
Device:Crystal_GND24 and wire the case pads to GND. Both 4-pad crystal
footprints put the terminals on pads 1/3 and the case on 2/4, so pins 1
and 3 keep their existing positions and the XTAL wiring is untouched.

D-sub shell (J8, J9). Move to DE15_Socket_HighDensity_MountingHoles,
whose pins 1-15 sit exactly where the old symbol's did, and rename the
footprint's two shell pads to SH. The shells now tie to GND, which is
the usual default; if the shells should instead be isolated from signal
ground, revert this part.

Verified by cross-checking every symbol's pins against its footprint's
pads across all sheets: no unmatched pads remain. Netlists confirm
U5.2/U7.2, Y2.2/Y2.4 and J8.SH/J9.SH all sit on GND.

Co-Authored-By: Claude Opus 5 <noreply@anthropic.com>
Claude-Session: https://claude.ai/code/session_01Ej9hevrS5JU2uwVi6UHQUS
Parts:
- J8, J9: symbol Connector:DE15_Socket_HighDensity -> Connector:DE15_Socket_HighDensity_MountingHoles
Connections:
- net GND: now also J8.SH, J9.SH
Changed lines of the file:
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@@
 	)
 	(symbol
-		(lib_id "Connector:DE15_Socket_HighDensity")
+		(lib_id "Connector:DE15_Socket_HighDensity_MountingHoles")
 		(at 188.214 261.366 0)
 		(unit 1)
@@
 		(pin "4"
 		)
+		(pin "SH"
+		)
 		(instances
 			(project "DegraderDosimeter"
@@
 	)
 	(symbol
-		(lib_id "Connector:DE15_Socket_HighDensity")
+		(lib_id "Connector:DE15_Socket_HighDensity_MountingHoles")
 		(at 92.964 261.62 0)
 		(unit 1)
@@
 		(pin "4"
 		)
+		(pin "SH"
+		)
 		(instances
 			(project "DegraderDosimeter"
@@
 					(unit 1)
 				)
+			)
+		)
+	)
+	(wire
+		(pts
+			(xy 92.964 279.400) (xy 92.964 281.940)
+		)
+		(stroke
+			(width 0)
+			(type default)
+		)
+	)
+	(symbol
+		(lib_id "power:GND")
+		(at 92.964 281.940 0)
+		(unit 1)
+		(body_style 1)
+		(exclude_from_sim no)
+		(in_bom yes)
+		(on_board yes)
+		(in_pos_files yes)
+		(dnp no)
+		(fields_autoplaced yes)
+		(property "Reference" "#PWR0201"
+			(at 92.964 280.940 0)
+			(hide yes)
+			(show_name no)
+			(do_not_autoplace no)
+			(effects
+				(font
+					(size 1.27 1.27)
+				)
+			)
+		)
+		(property "Value" "GND"
+			(at 92.964 285.140 0)
+			(show_name no)
+			(do_not_autoplace no)
+			(effects
+				(font
+					(size 1.27 1.27)
+				)
+			)
+		)
+		(pin "1"
+		)
+		(instances
+			(project "DegraderDosimeter"
+				(path "/f3c83d46-b432-4960-ae55-27eb620ca6d0/9ad00133-e13c-465e-ad59-297593e6d3f6"
+					(reference "#PWR0201")
+					(unit 1)
+				)
+			)
+		)
+	)
+	(wire
+		(pts
+			(xy 188.214 279.146) (xy 188.214 281.686)
+		)
+		(stroke
+			(width 0)
+			(type default)
+		)
+	)
+	(symbol
+		(lib_id "power:GND")
+		(at 188.214 281.686 0)
+		(unit 1)
+		(body_style 1)
+		(exclude_from_sim no)
+		(in_bom yes)
+		(on_board yes)
+		(in_pos_files yes)
+		(dnp no)
+		(fields_autoplaced yes)
+		(property "Reference" "#PWR0202"
+			(at 188.214 280.686 0)
+			(hide yes)
+			(show_name no)
+			(do_not_autoplace no)
+			(effects
+				(font
+					(size 1.27 1.27)
+				)
+			)
+		)
+		(property "Value" "GND"
+			(at 188.214 284.886 0)
+			(show_name no)
+			(do_not_autoplace no)
+			(effects
+				(font
+					(size 1.27 1.27)
+				)
+			)
+		)
+		(pin "1"
+		)
+		(instances
+			(project "DegraderDosimeter"
+				(path "/f3c83d46-b432-4960-ae55-27eb620ca6d0/9ad00133-e13c-465e-ad59-297593e6d3f6"
+					(reference "#PWR0202")
+					(unit 1)
+				)
