File: Schematics/DegraderDosimeter/MCU_H723.kicad_sch (KiCad schematic)
At the start: 25 parts, among them SW1 SW_Push_Dual_x2, U5 STM32H723ZGTx, Y2 Crystal

Commit message: Set MCU ferrite bead to the MB1364 BOM part
FB2, on the VDD to VDDA feed, carried the placeholder value
"FerriteBead_Small" and a through-hole footprint
(Ferrite_THT:LairdTech_28C0236-0JW-10) on an otherwise all-SMD board.

Assign the only ferrite bead in the MB1364-H723ZG-E01 BOM, TAI-TECH
FCM1608KF-601T03 (600R@100MHz +/-25%, 350mA, 500mohm DC, 0603), so both
ferrites on the design share one part number.

Note this is a deliberate deviation from the Nucleo: MB1364 feeds VDDA
through R37, a 0R 0603 resistor, and fits no ferrite there at all. The
bead is kept for VDDA supply filtering.

ERC violation count is unchanged at 1445.

Co-Authored-By: Claude Opus 5 <noreply@anthropic.com>
Claude-Session: https://claude.ai/code/session_01Ej9hevrS5JU2uwVi6UHQUS
Parts:
- FB2: value FerriteBead_Small -> 600R@100MHz; footprint Ferrite_THT:LairdTech_28C0236-0JW-10 -> Inductor_SMD:L_0603_1608Metric

Commit message: Use 1206 for every resistor in the project
The Ethernet sheet was the only one on 0402, set that way to match the
MB1364 BOM. The other four sheets already used
Resistor_SMD:R_1206_3216Metric_Pad1.30x1.75mm_HandSolder, so move the
20 Ethernet resistors to the same footprint. All 37 resistors in the
project now share one package, which suits hand assembly.

This deviates from the ST reference for the eight resistors on the
high-speed nets: R3-R6 (33R RMII series) and R12-R15 (49R9 centre-tap
terminations). 1206 has more parasitic inductance and larger pads than
the 0402 parts ST fits. 100BASE-TX is tolerant enough that this should
still work, but 0402 would be the better choice on those eight.

This commit also captures schematic edits made in KiCad outside this
session: a project-wide re-annotation and the removal of R21/R22, the
two 75R resistors that terminated the jack's unused pairs.

Co-Authored-By: Claude Opus 5 <noreply@anthropic.com>
Claude-Session: https://claude.ai/code/session_01Ej9hevrS5JU2uwVi6UHQUS
Parts:
- renumbered C53 to C11, C54 to C12, C12 to C13, C39 to C14, C38 to C15, C56 to C16, C55 to C17, C52 to C18, C40 to C19, C44 to C20, C48 to C21, C41 to C22, C45 to C23, C49 to C24, C42 to C25, C46 to C26, C50 to C27, C43 to C28, C47 to C29, C51 to C30, R58 to R21, U5 to U4

Commit message: Give every footprint pad a symbol pin so no pad is left netless
Updating the PCB warned about eight pads that had no matching symbol
pin, so they would have been placed with no net: U5/U7 pad 4, Y2 pads
3 and 4, and J8/J9 pads 16 and 17. Three separate causes:

SOT-223 tab (U5, U7). The TC1262 tab is electrically the same node as
pin 2, GND; the vendor symbol in Libs/TC1262-3.3VDB draws pins 2 and 4
stacked at one point, which confirms it. Renumber the footprint's tab
pad from 4 to 2 so it inherits GND. No schematic change, and the tab is
the regulator's heat path, so it needs to be connected.

Crystal case (Y2). Same fix already applied to Y1: Device:Crystal on a
4-pad footprint left the two case pads unmapped. Move to
Device:Crystal_GND24 and wire the case pads to GND. Both 4-pad crystal
footprints put the terminals on pads 1/3 and the case on 2/4, so pins 1
and 3 keep their existing positions and the XTAL wiring is untouched.

D-sub shell (J8, J9). Move to DE15_Socket_HighDensity_MountingHoles,
whose pins 1-15 sit exactly where the old symbol's did, and rename the
footprint's two shell pads to SH. The shells now tie to GND, which is
the usual default; if the shells should instead be isolated from signal
ground, revert this part.

Verified by cross-checking every symbol's pins against its footprint's
pads across all sheets: no unmatched pads remain. Netlists confirm
U5.2/U7.2, Y2.2/Y2.4 and J8.SH/J9.SH all sit on GND.

Co-Authored-By: Claude Opus 5 <noreply@anthropic.com>
Claude-Session: https://claude.ai/code/session_01Ej9hevrS5JU2uwVi6UHQUS
Parts:
- Y2: symbol Device:Crystal -> Device:Crystal_GND24
Connections:
- net GND: now also Y2.2 (G), Y2.4 (G)
- net at C12.2, U4.23 (PH0): now also Y2.3; no longer Y2.2
