File: Schematics/DegraderDosimeter/MCU_H723.kicad_sch (KiCad schematic)
At the start: 25 parts, among them SW1 SW_Push_Dual_x2, U5 STM32H723ZGTx, Y2 Crystal

Commit message: Bring the DegraderDosimeter schematic up to a routable state
Single ECAD commit on top of "First upload", carrying both the earlier
board-bring-up work and this session's changes. Squashed here so the
schematic history is separate from the FirmwareUpdate restructure, which
stays on main.

Library resolution
  Register the A4988 and LM60430DRPKR symbol libraries in sym-lib-table,
  and the DE15, DRIVER-A4988SETTR-T_QFN28_ and KRJ-CB4.2GYZNL footprint
  libraries in fp-lib-table. Point H1102NL at ${KIPRJMOD} instead of the
  undefined ${CUSTOM}. All 26 symbols and 24 footprints now resolve.

Degrader to MCU
  Wire all 32 degrader signals to the STM32H723: 11 A4988/L293D controls
  and 21 lens limit switches. Reuse the F746 firmware's pin assignment
  where it does not clash with the dosimeter; MS1 and MS2 move to PD14
  and PD15 because PD11/PD12 are pulse-capture pins, and !ENABLE takes
  PB7 as the firmware never assigned it. Grow the MCU_H723 sheet so its
  right edge spans the Degrader sheet, giving one straight wire per net.

Net naming and classes
  Drop the duplicate port label on the 50 pins that already carry a
  functional hierarchical label, so nets read STEP/MS1/RMII_REF_CLK
  rather than PD14/PA1; unused pins keep their port label and bus. Name
  the remaining 73 auto-named nets. Add ETH_DIFF_100R, ETH_RMII, POWER,
  MOTOR and ANALOG net classes. The four MDI pairs get 0.15 mm track on
  a 0.30 mm gap, which is 100 ohm differential on the declared stackup
  (F.Cu over In1.Cu, 0.1 mm prepreg, er 4.5) - reconfirm if the fab
  ships a different stackup.

Connection fixes
  - MDC/MDIO were crossed: PA2 landed on the PHY's MDC pin and PC1 on
    MDIO. Swapped the two labels in Ethernet.kicad_sch.
  - PULSE_6 moved PD11 -> PD12, the TIM4_CH1 pin BLM_Code.ioc expects.
  - PulseShaper 1, 2 and 5 outputs missed their sheet pins by 2-81 um.
  - XTAL1 stopped 0.254 mm short of Y1/C1, leaving the PHY crystal open.
  - C32/C35 and C39/C40, the U5 and U7 cap returns, h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
Parts:
- FB2: value FerriteBead_Small -> 600R@100MHz; footprint Ferrite_THT:LairdTech_28C0236-0JW-10 -> Inductor_SMD:L_0603_1608Metric
- Y2: symbol Device:Crystal -> Device:Crystal_GND24
- renumbered C53 to C11, C54 to C12, C12 to C13, C39 to C14, C38 to C15, C56 to C16, C55 to C17, C52 to C18, C40 to C19, C44 to C20, C48 to C21, C41 to C22, C45 to C23, C49 to C24, C42 to C25, C46 to C26, C50 to C27, C43 to C28, C47 to C29, C51 to C30, R58 to R21, U5 to U4
Connections:
- net PD12 is gone; now on net PULSE_6: U4.81 (PD12)
- net GND: now also Y2.2 (G), Y2.4 (G)
- net PULSE_6: no longer U4.80 (PD11)
- net VCAP2: now reaches C15.1, U4.106 (VCAP)
- net HSE_IN: now reaches C12.2, U4.23 (PH0)
- net HSE_IN: now also Y2.3; no longer Y2.2
- net HSE_OUT: now reaches C11.2, U4.24 (PH1), Y2.1
- net NRST: now reaches C14.2, SW1.1 (C), U4.25 (NRST)
- net VBAT: now reaches C16.1, U4.6 (VBAT)
- net VCAP1: now reaches C13.1, U4.71 (VCAP)
- net PA3 renamed 3mm_LEFT_SWITCH
- net PB14 renamed STEP
- net PB2 renamed !RESET
- net PB5 renamed DC_MOTOR_EN
- net PB6 renamed !SLEEP
- net PB7 renamed !ENABLE
- net PC0 renamed 12mm_SELECTED_SWITCH
- net PC2 renamed DIR
- net PC3 renamed 30mm_SELECTED_SWITCH
- net PC6 renamed DC_MOTOR_DIR2
- net PC7 renamed DC_MOTOR_DIR1
- net PD0 renamed 10mm_LEFT_SWITCH
- net PD1 renamed 2mm_LEFT_SWITCH
- net PD13 renamed MS3
- net PD14 renamed MS1
- net PD15 renamed MS2
- net PD3 renamed 2mm_SELECTED_SWITCH
- net PD4 renamed 10mm_RIGHT_SWITCH
- net PD5 renamed 30mm_RIGHT_SWITCH
- net PD6 renamed 12mm_RIGHT_SWITCH
- net PD7 renamed 6mm_LEFT_SWITCH
- net PE2 renamed 3mm_RIGHT_SWITCH
- net PE3 renamed 30mm_LEFT_SWITCH
- net PE4 renamed 6mm_RIGHT_SWITCH
- net PE5 renamed 2mm_RIGHT_SWITCH
- net PE6 renamed 8mm_RIGHT_SWITCH
- net PF10 renamed 12mm_LEFT_SWITCH
- net PF2 renamed 10mm_SELECTED_SWITCH
- net PF3 renamed 6mm_SELECTED_SWITCH
- net PF5 renamed 8mm_LEFT_SWITCH
- net PF7 renamed 8mm_SELECTED_SWITCH
- net PF8 renamed 3mm_SELECTED_SWITCH
- new net PD11: U4.80 (PD11)
