File: Schematics/DegraderDosimeter/MCU_H723.kicad_sch (KiCad schematic)
At the start: 25 parts, among them SW1 SW_Push_Dual_x2, U4 STM32H723ZGTx, Y2 Crystal

Commit message: Update: Combine degrader and dosimeter schematics
Parts:
- C11, C12, C13, C15: footprint Capacitor_SMD:C_1206_3216Metric -> Capacitor_SMD:C_0603_1608Metric
- C14, C17, C19, C20, C21, C22, C23, C24, C25, C26, C27, C28, C29, C30: footprint Capacitor_SMD:C_1206_3216Metric -> Capacitor_SMD:C_0603_1608Metric; LCSC (none) -> C14663
- C16: footprint Capacitor_SMD:C_1206_3216Metric -> Capacitor_SMD:C_0603_1608Metric; LCSC (none) -> C15849
- C18: footprint Capacitor_SMD:C_1206_3216Metric -> Capacitor_SMD:C_0603_1608Metric; LCSC (none) -> C19666
- R21: footprint Resistor_SMD:R_1206_3216Metric_Pad1.30x1.75mm_HandSolder -> Resistor_SMD:R_0603_1608Metric; LCSC (none) -> C25804
- SW1: now not fitted
Connections:
- net PB10 renamed ST_STEP2
- net PB11 renamed ST_DIR2
- net PB12 renamed !ST_EN2
- net PB15 renamed !ADC_ALERT
- net PB8 renamed I2C1_SCL
- net PB9 renamed I2C1_SDA
- net PC10 renamed !ST_EN3
- net PC8 renamed ST_STEP3
- net PC9 renamed ST_DIR3
- net PE10 renamed ST_DIR1
- net PE11 renamed !ST_EN1
- net PE12 renamed ST_MS1
- net PE13 renamed ST_MS2
- net PE14 renamed ST_MS3
- net PE15 renamed !ST_RESET
- net PE9 renamed ST_STEP1
- net PG0 renamed !ST_SLEEP
