File: Schematics/DegraderDosimeter/Power_supply.kicad_sch (KiCad schematic)
At the start: 25 parts, among them U4 LM60430DRPKR, U6 TC1262-33, U7 TC1262-33

Commit message: Bring the DegraderDosimeter schematic up to a routable state
Single ECAD commit on top of "First upload", carrying both the earlier
board-bring-up work and this session's changes. Squashed here so the
schematic history is separate from the FirmwareUpdate restructure, which
stays on main.

Library resolution
  Register the A4988 and LM60430DRPKR symbol libraries in sym-lib-table,
  and the DE15, DRIVER-A4988SETTR-T_QFN28_ and KRJ-CB4.2GYZNL footprint
  libraries in fp-lib-table. Point H1102NL at ${KIPRJMOD} instead of the
  undefined ${CUSTOM}. All 26 symbols and 24 footprints now resolve.

Degrader to MCU
  Wire all 32 degrader signals to the STM32H723: 11 A4988/L293D controls
  and 21 lens limit switches. Reuse the F746 firmware's pin assignment
  where it does not clash with the dosimeter; MS1 and MS2 move to PD14
  and PD15 because PD11/PD12 are pulse-capture pins, and !ENABLE takes
  PB7 as the firmware never assigned it. Grow the MCU_H723 sheet so its
  right edge spans the Degrader sheet, giving one straight wire per net.

Net naming and classes
  Drop the duplicate port label on the 50 pins that already carry a
  functional hierarchical label, so nets read STEP/MS1/RMII_REF_CLK
  rather than PD14/PA1; unused pins keep their port label and bus. Name
  the remaining 73 auto-named nets. Add ETH_DIFF_100R, ETH_RMII, POWER,
  MOTOR and ANALOG net classes. The four MDI pairs get 0.15 mm track on
  a 0.30 mm gap, which is 100 ohm differential on the declared stackup
  (F.Cu over In1.Cu, 0.1 mm prepreg, er 4.5) - reconfirm if the fab
  ships a different stackup.

Connection fixes
  - MDC/MDIO were crossed: PA2 landed on the PHY's MDC pin and PC1 on
    MDIO. Swapped the two labels in Ethernet.kicad_sch.
  - PULSE_6 moved PD11 -> PD12, the TIM4_CH1 pin BLM_Code.ioc expects.
  - PulseShaper 1, 2 and 5 outputs missed their sheet pins by 2-81 um.
  - XTAL1 stopped 0.254 mm short of Y1/C1, leaving the PHY crystal open.
  - C32/C35 and C39/C40, the U5 and U7 cap returns, h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
Parts:
- U6: renamed from U4; footprint RPK0013A-MFG -> RPK0013A-MFG:RPK0013A-MFG
- renumbered C11 to C31, C22 to C32, C13 to C33, C14 to C34, C23 to C35, C15 to C36, C16 to C37, C21 to C38, C24 to C39, C25 to C40, C20 to C41, C19 to C42, C18 to C43, C17 to C44, L2 to L1, L1 to L2, R24 to R22, R27 to R24, U6 to U5
Connections:
- net GND: now also C32.2, C35.2, C39.2, C40.2, C44.2, R26.1
- net VCC: now also L1.1
- net VIN_FLT2: now reaches R22.2
- net VIN_FLT2: now also C31.1, L1.2, L2.1; no longer L1.1
- net BUCK_VIN_DAMP: now reaches C33.1, R23.2
- net BUCK_FB: now reaches C42.2, R25.1, R26.2, U6.7 (FB)
- net BUCK_BOOT: now reaches C41.1, U6.4 (BOOT)
- net BUCK_SW: now reaches C41.2, L3.1, U6.12 (SW)
- net BUCK_VIN: now reaches C34.1, C36.1, C37.1, L2.2, R23.1, U6.10 (VIN), U6.2 (VIN), U6.9 (EN)
- net BUCK_VCC: now reaches C38.1, U6.5 (VCC)
- net BUCK_PG: now reaches R24.2, U6.8 (PG)
Other:
- moved on the sheet: R22
