File: Schematics/DegraderDosimeter/DegraderDosimeter.kicad_sch (KiCad schematic)
At the start: 0 parts

Commit message: Update: Combine degrader and dosimeter schematics
Other:
- added sheet ADC_I2C (ADC_I2C.kicad_sch)
- added sheet Debugger (Debugger.kicad_sch)
- added sheet MotorSupply (MotorSupply.kicad_sch)
- added sheet StepperDrivers (StepperDrivers.kicad_sch)
- sheet MCU_H723 ports: added !ADC_ALERT, !ST_EN1, !ST_EN2, !ST_EN3, !ST_RESET, !ST_SLEEP, I2C1_SCL, I2C1_SDA, ST_DIR1, ST_DIR2, ST_DIR3, ST_MS1, ST_MS2, ST_MS3, ST_STEP1, ST_STEP2, ST_STEP3; removed none
